Commit message: Add 360 degree LiDAR with shared sensor mast placement

File: src/porter_description/urdf/chassis.xacro (robot description, xacro)
@@ -24,4 +24,10 @@
   <xacro:property name="wheel_dy"       value="${chassis_width/2 + wheel_width/2}"/>
   <xacro:property name="wheel_separation" value="${2*wheel_dy}"/>
+  <!-- Sensor mast position. The LiDAR and the camera share this X so that a
+       bearing measured by the camera can be used directly as a LiDAR ray
+       index. Both lidar.xacro and camera.xacro read it from here. -->
+  <xacro:property name="sensor_mast_x"  value="0.26"/>
+  <xacro:property name="lidar_height"   value="0.25"/>
+  <xacro:property name="camera_height"  value="1.00"/>
   <xacro:property name="platform_length" value="0.50"/>
   <xacro:property name="platform_width"  value="0.40"/>

File: src/porter_description/urdf/porter.urdf.xacro (robot description, xacro)
@@ -5,6 +5,6 @@
 <robot name="porter" xmlns:xacro="http://www.ros.org/wiki/xacro">
   <xacro:include filename="$(find porter_description)/urdf/chassis.xacro"/>
+  <xacro:include filename="$(find porter_description)/urdf/lidar.xacro"/>
   <!-- Sensors are added as they are implemented:
-       <xacro:include filename="$(find porter_description)/urdf/lidar.xacro"/>
        <xacro:include filename="$(find porter_description)/urdf/camera.xacro"/>
        <xacro:include filename="$(find porter_description)/urdf/imu.xacro"/> -->

Commit message: Enlarge chassis, add caster struts and move LiDAR to the front bumper

File: src/porter_description/urdf/chassis.xacro (robot description, xacro)
@@ -5,17 +5,17 @@
 <robot xmlns:xacro="http://www.ros.org/wiki/xacro">
   <!-- ============================ Dimensions ============================ -->
-  <xacro:property name="chassis_length" value="0.60"/>
-  <xacro:property name="chassis_width"  value="0.45"/>
-  <xacro:property name="chassis_height" value="0.12"/>
-  <xacro:property name="chassis_mass"   value="15.0"/>
-  <xacro:property name="wheel_radius"   value="0.08"/>
-  <xacro:property name="wheel_width"    value="0.04"/>
-  <xacro:property name="wheel_mass"     value="1.5"/>
-  <xacro:property name="caster_radius"  value="0.04"/>
+  <xacro:property name="chassis_length" value="0.75"/>
+  <xacro:property name="chassis_width"  value="0.55"/>
+  <xacro:property name="chassis_height" value="0.15"/>
+  <xacro:property name="chassis_mass"   value="22.0"/>
+  <xacro:property name="wheel_radius"   value="0.11"/>
+  <xacro:property name="wheel_width"    value="0.05"/>
+  <xacro:property name="wheel_mass"     value="2.2"/>
+  <xacro:property name="caster_radius"  value="0.035"/>
   <xacro:property name="caster_mass"    value="0.3"/>
-  <xacro:property name="caster_offset"  value="0.25"/>   <!-- +-X from centre -->
+  <xacro:property name="caster_offset"  value="0.31"/>   <!-- +-X from centre -->
   <!-- Chassis centre height. The wheel axle must sit exactly one wheel radius
        above the ground, so the wheel joints are lowered by this difference. -->
-  <xacro:property name="base_height"    value="0.14"/>
+  <xacro:property name="base_height"    value="0.20"/>
   <xacro:property name="wheel_dz"       value="${wheel_radius - base_height}"/>
   <xacro:property name="caster_dz"      value="${caster_radius - base_height}"/>
@@ -24,12 +24,16 @@
   <xacro:property name="wheel_dy"       value="${chassis_width/2 + wheel_width/2}"/>
   <xacro:property name="wheel_separation" value="${2*wheel_dy}"/>
-  <!-- Sensor mast position. The LiDAR and the camera share this X so that a
-       bearing measured by the camera can be used directly as a LiDAR ray
-       index. Both lidar.xacro and camera.xacro read it from here. -->
-  <xacro:property name="sensor_mast_x"  value="0.26"/>
+  <!-- Sensor placement, shared by lidar.xacro and camera.xacro.
+       Both sensors sit on the SAME vertical axis (sensor_x) so that a bearing
+       measured in the image maps directly onto a LiDAR ray index with no
+       parallax correction. The supporting post stands further back at
+       mast_post_x and carries the camera forward on a short arm, which keeps
+       it out of the LiDAR scan plane. -->
+  <xacro:property name="sensor_x"       value="0.41"/>
+  <xacro:property name="mast_post_x"    value="0.33"/>
   <xacro:property name="lidar_height"   value="0.25"/>
   <xacro:property name="camera_height"  value="1.00"/>
-  <xacro:property name="platform_length" value="0.50"/>
-  <xacro:property name="platform_width"  value="0.40"/>
+  <xacro:property name="platform_length" value="0.62"/>
+  <xacro:property name="platform_width"  value="0.48"/>
   <xacro:property name="platform_thick"  value="0.02"/>
   <xacro:property name="rail_height"     value="0.06"/>
@@ -94,4 +98,8 @@
   <!-- One caster, modelled as a frictionless sphere rigidly attached to the
        body. A real swivel joint is unnecessary and only adds instability. -->
+  <xacro:property name="caster_strut_radius" value="0.013"/>
+  <!-- Leg from the chassis underside down to the top of the ball. -->
+  <xacro:property name="caster_strut_length"
+                  value="${base_height - chassis_height/2 - 2*caster_radius}"/>
   <xacro:macro name="caster" params="prefix side">
     <link name="${prefix}_caster_link">
@@ -99,4 +107,12 @@
         <geometry><sphere radius="${caster_radius}"/></geometry>
         <material name="porter_dark"/>
+      </visual>
+      <!-- Thin leg, drawn upwards from the ball to the chassis. -->
+      <visual>
+        <origin xyz="0 0 ${caster_radius + caster_strut_length/2}" rpy="0 0 0"/>
+        <geometry>
+          <cylinder radius="${caster_strut_radius}" length="${caster_strut_length}"/>
+        </geometry>
+        <material name="porter_accent"/>
       </visual>
       <collision>
@@ -189,4 +205,7 @@
             name="gz::sim::systems::JointStatePublisher">
       <topic>joint_states</topic>
+      <!-- Without a rate limit this publishes at the physics step rate
+           (~1000 Hz), which is far more than RViz needs. -->
+      <update_rate>50</update_rate>
     </plugin>
   </gazebo>

File: src/porter_description/urdf/lidar.xacro (robot description, xacro)
@@ -7,8 +7,4 @@
   <xacro:property name="lidar_length" value="0.045"/>
   <xacro:property name="lidar_mass"   value="0.17"/>
-  <!-- The post runs from the chassis top up to the underside of the puck. -->
-  <xacro:property name="post_radius"  value="0.012"/>
-  <xacro:property name="chassis_top"  value="${base_height + chassis_height/2}"/>
-  <xacro:property name="post_length"  value="${lidar_height - lidar_length/2 - chassis_top}"/>
   <link name="lidar_link">
     <!-- Sensor body. Its origin is the measurement origin, so the scan
@@ -17,10 +13,4 @@
       <geometry><cylinder radius="${lidar_radius}" length="${lidar_length}"/></geometry>
       <material name="porter_dark"/>
-    </visual>
-    <!-- Support post, drawn downwards from the puck to the chassis. -->
-    <visual>
-      <origin xyz="0 0 ${-lidar_length/2 - post_length/2}" rpy="0 0 0"/>
-      <geometry><cylinder radius="${post_radius}" length="${post_length}"/></geometry>
-      <material name="porter_accent"/>
     </visual>
     <collision>
@@ -37,5 +27,5 @@
     <parent link="base_link"/>
     <child  link="lidar_link"/>
-    <origin xyz="${sensor_mast_x} 0 ${lidar_height - base_height}" rpy="0 0 0"/>
+    <origin xyz="${sensor_x} 0 ${lidar_height - base_height}" rpy="0 0 0"/>
   </joint>
   <gazebo reference="lidar_link">
@@ -49,10 +39,17 @@
       <frame_id>lidar_link</frame_id>
       <lidar>
+        <!-- Front mounted, so the rear arc is blocked by the chassis anyway.
+             The chassis corners block the view beyond +-97 degrees, so the
+             scan is limited to +-90 with a small margin: every returned ray
+             is real. 181 samples give one degree per ray. The camera only
+             sees +-40 degrees, so the target bearing always falls inside.
+             The controller needs the target bearing and the forward +-30
+             degrees, both well inside this field. -->
         <scan>
           <horizontal>
-            <samples>360</samples>
+            <samples>181</samples>
             <resolution>1</resolution>
-            <min_angle>${-pi}</min_angle>
-            <max_angle>${pi}</max_angle>
+            <min_angle>${-pi/2}</min_angle>
+            <max_angle>${ pi/2}</max_angle>
           </horizontal>
         </scan>

Commit message: Move both casters ahead of the drive wheels so the robot climbs the ramp
Porter could not get up the 8 degree ramp. Driven straight at it with no
controller in the loop it veered 1.3 m sideways and slid off the ramp's edge;
through the shared launch it stopped partway up and stayed there. Nine
simulation runs isolated the cause.

The casters sat one at each end, 0.62 m apart, with the drive wheels at the
midpoint. Straddling the foot of the ramp, the rigid chassis follows the
straight line between the two caster contacts, and that lifts the mid-mounted
wheels clear of the surface: 2.2 cm on an 8 degree slope. The wheels then turn
at the commanded rate against nothing. The measured body pitch of 4.35 degrees
matches the 4.03 degrees this geometry predicts.

Three explanations were ruled out, each by measurement rather than argument:

- Ramp angle. At 6 and 4 degrees the robot fails the same way, drifting 1.36
  and 1.34 m. A longer, shallower ramp was the mitigation the project document
  proposed for this risk, and it does not work.
- Caster friction. At mu 0.6 and 1.2 the drift disappears but the robot cannot
  get onto the ramp at all. Only the failure mode changes.
- Wheel position on its own. Moving the axle back 0.18 m while keeping a caster
  at each end still drifts 1.40 m. The wheels are always between the casters,
  so moving them cannot help; this run was made to falsify that prediction and
  did not.

Both casters now sit ahead of the wheels as a lateral pair at x 0.31, y +-0.18,
and the axle moves 0.10 m behind the centre of mass. The pair alone fixes the
climb. The axle offset is what makes it safe: with the mass straight over the
axle the body rocks 19 degrees nose-up under acceleration, with nothing behind
it to catch the body. With both changes the robot climbs the ramp and crosses
the deck with 7 mm of lateral drift, and pitches 0.00 degrees under both
acceleration and braking.

Through the full launch it now follows the person over the whole route, holding
0.897 to 1.316 m against a 1.000 m set point, climbs the ramp, and settles
0.963 m behind the person once they stop.

One consequence worth stating: base_link no longer coincides with the point the
robot turns about, so the drive plugin's odometry refers to the axle, 0.10 m
behind it. The following behaviour does not read odometry. The swept turning
diameter grows from 0.93 m to 1.10 m, inside the 1.4 m aisles of the world.

File: src/porter_description/urdf/chassis.xacro (robot description, xacro)
@@ -14,5 +14,18 @@
   <xacro:property name="caster_radius"  value="0.035"/>
   <xacro:property name="caster_mass"    value="0.3"/>
-  <xacro:property name="caster_offset"  value="0.31"/>   <!-- +-X from centre -->
+  <!-- Both casters sit ahead of the drive wheels, as a lateral pair, and never
+       one at each end. Casters fore and aft straddle the foot of a ramp, and
+       the rigid chassis then follows the straight line between them, lifting
+       the drive wheels clear of the surface: 2.2 cm on the 8 degree ramp,
+       which is enough to lose traction entirely. -->
+  <xacro:property name="caster_x"       value="0.31"/>
+  <xacro:property name="caster_dy"      value="0.18"/>   <!-- +-Y of the pair -->
+  <!-- The axle sits behind the centre of mass, so the body always leans onto
+       the casters. With the axle under the centre of mass the robot rocks
+       about 19 degrees nose-up under acceleration, with nothing behind it to
+       catch the body. Note that base_link therefore no longer coincides with
+       the point the robot turns about: odometry from the drive plugin refers
+       to the axle, 0.10 m behind base_link. -->
+  <xacro:property name="wheel_x"        value="-0.10"/>
   <!-- Chassis centre height. The wheel axle must sit exactly one wheel radius
        above the ground, so the wheel joints are lowered by this difference. -->
@@ -87,5 +100,5 @@
       <parent link="base_link"/>
       <child  link="${prefix}_wheel_link"/>
-      <origin xyz="0 ${side*wheel_dy} ${wheel_dz}" rpy="0 0 0"/>
+      <origin xyz="${wheel_x} ${side*wheel_dy} ${wheel_dz}" rpy="0 0 0"/>
       <axis xyz="0 1 0"/>
     </joint>
@@ -96,6 +109,7 @@
     </gazebo>
   </xacro:macro>
-  <!-- One caster, modelled as a frictionless sphere rigidly attached to the
-       body. A real swivel joint is unnecessary and only adds instability. -->
+  <!-- One caster of the front pair, modelled as a frictionless sphere rigidly
+       attached to the body. A real swivel joint is unnecessary and only adds
+       instability; side selects the left or right of the pair. -->
   <xacro:property name="caster_strut_radius" value="0.013"/>
   <!-- Leg from the chassis underside down to the top of the ball. -->
@@ -124,5 +138,5 @@
       <parent link="base_link"/>
       <child  link="${prefix}_caster_link"/>
-      <origin xyz="${side*caster_offset} 0 ${caster_dz}" rpy="0 0 0"/>
+      <origin xyz="${caster_x} ${side*caster_dy} ${caster_dz}" rpy="0 0 0"/>
     </joint>
     <gazebo reference="${prefix}_caster_link">
@@ -182,6 +196,6 @@
   <xacro:drive_wheel prefix="left"  side="1"/>
   <xacro:drive_wheel prefix="right" side="-1"/>
-  <xacro:caster      prefix="front" side="1"/>
-  <xacro:caster      prefix="rear"  side="-1"/>
+  <xacro:caster      prefix="front_left"  side="1"/>
+  <xacro:caster      prefix="front_right" side="-1"/>
   <!-- ============================= Gazebo =============================== -->
   <gazebo>

Commit message: Put a visible load on the cargo deck
Porter's job is to carry something, and until now the deck was empty, so
neither the simulation nor the demonstration video showed what the robot is
for. Add a crate, a box stacked on it and a parcel alongside.

These are visual elements on the existing deck link, not a new link and not
new mass. The drive axle is deliberately set 0.10 m behind the centre of mass
so the body leans onto the front casters; giving the load mass would move that
centre and undo it. The generated model is unchanged where it matters: 13
links, 12 joints, 9 collision shapes and 29.790 kg before and after, with only
the visual count rising from 16 to 19.

The crates sit above the LiDAR's scan plane and behind the camera, so neither
sensor can see them.

File: src/porter_description/urdf/chassis.xacro (robot description, xacro)
@@ -52,8 +52,19 @@
   <xacro:property name="rail_height"     value="0.06"/>
   <xacro:property name="rail_thick"      value="0.015"/>
+  <!-- The load Porter carries. Visual only, like the deck it sits on: the
+       robot's job has to be readable at a glance in the simulation and in the
+       demonstration video. Giving it mass would move the centre of mass that
+       the axle offset is set against (see the drive wheel section), so the
+       crates deliberately carry none. They sit above the LiDAR plane and
+       behind the camera, so neither sensor sees them. -->
+  <xacro:property name="crate_a" value="0.34 0.30 0.26"/>   <!-- lower crate -->
+  <xacro:property name="crate_b" value="0.22 0.20 0.16"/>   <!-- stacked box -->
+  <xacro:property name="crate_c" value="0.20 0.26 0.20"/>   <!-- parcel beside -->
   <!-- ============================= Materials ============================ -->
   <material name="porter_body">  <color rgba="0.15 0.35 0.55 1"/></material>
   <material name="porter_dark">  <color rgba="0.15 0.15 0.17 1"/></material>
   <material name="porter_accent"><color rgba="0.85 0.85 0.88 1"/></material>
+  <material name="porter_crate"> <color rgba="0.55 0.40 0.25 1"/></material>
+  <material name="porter_parcel"><color rgba="0.30 0.33 0.38 1"/></material>
   <!-- ============================== Macros ============================== -->
   <!-- Solid box inertia about its own centre. -->
@@ -164,6 +175,7 @@
                        y="${chassis_width}" z="${chassis_height}"/>
   </link>
-  <!-- Cargo deck with low rails. Visual only: it carries no load in
-       simulation and collision shapes here would only slow physics down. -->
+  <!-- Cargo deck with low rails, and the load it carries. Visual only:
+       collision shapes here would only slow physics down, and mass here would
+       shift the centre of mass the drive axle is positioned against. -->
   <link name="cargo_deck_link">
     <visual>
@@ -185,4 +197,22 @@
       <geometry><box size="${rail_thick} ${platform_width} ${rail_height}"/></geometry>
       <material name="porter_accent"/>
+    </visual>
+    <!-- Cargo: a crate with a box stacked on it, and a parcel alongside.
+         Each sits on the deck plate, so its centre is half its own height
+         above the top face. -->
+    <visual>
+      <origin xyz="-0.10 0 ${platform_thick/2 + 0.13}"/>
+      <geometry><box size="${crate_a}"/></geometry>
+      <material name="porter_crate"/>
+    </visual>
+    <visual>
+      <origin xyz="-0.10 0 ${platform_thick/2 + 0.26 + 0.08}"/>
+      <geometry><box size="${crate_b}"/></geometry>
+      <material name="porter_parcel"/>
+    </visual>
+    <visual>
+      <origin xyz="0.18 0 ${platform_thick/2 + 0.10}"/>
+      <geometry><box size="${crate_c}"/></geometry>
+      <material name="porter_crate"/>
     </visual>
     <xacro:box_inertia m="2.0" x="${platform_length}"
